Commit message: add camera,multimachine,tebplanner

File: src/mobile_base_arm/urdf/mobile_base_arm.urdf (robot description, URDF)
Before this commit: robot mobile_base_arm, 21 links, 20 joints
Links:
- removed link MPU9250_fr
- added link MPU9250_fl, mass 0.00062885; collision mesh filename=package://mobile_base_arm/meshes/MPU9250_fl.STL; visual mesh filename=package://mobile_base_arm/meshes/MPU9250_fl.STL
- link base_link: mass 0.374892757850051 -> 0.31986
- link camera_link: mass 0 -> 0.0097885
Joints:
- removed joint MPU9250_fr_joint
- added joint MPU9250_fl_joint: type fixed, parent base_link, child MPU9250_fl, origin xyz=0.082311 0.072761 0.07357 rpy=0 0 0, axis 0 0 0
- joint bl_wheel_joint: origin xyz=-0.078453 0.14588 0.029654 rpy=1.5708 0 -3.1416 -> xyz=-0.078589 0.12644 0.029654 rpy=1.5708 0 -3.1416
- joint br_wheel_joint: origin xyz=-0.078453 -0.14712 0.029654 rpy=1.5708 0 0 -> xyz=-0.078589 -0.12656 0.029654 rpy=1.5708 0 0
- joint camera_joint: origin xyz=0.11165 -0.00061982 0.03 rpy=0 0 0 -> xyz=0.11151109677708 -5.58611123459007E-05 0.0299999999999999 rpy=0 0 0
- joint eef_finger_joint_1: origin xyz=-0.0250754321495898 0.0177984606781366 0.00134999999999999 rpy=0 0 0 -> xyz=-0.025075 0.017798 0.00135 rpy=0 0 0
- joint eef_joint_1: origin xyz=0.038466720887356 0.014139797883076 -0.0179 rpy=-1.5707963267949 0 3.10994225522667 -> xyz=0.038467 0.01414 -0.0179 rpy=-1.5708 0 3.1099
- joint eef_joint_2: origin xyz=0.038466720887356 0.014139797883076 0.00899999999999998 rpy=-1.5707963267949 0 3.10994225522667 -> xyz=0.038467 0.01414 0.009 rpy=-1.5708 0 3.1099
- joint fl_wheel_joint: origin xyz=0.078747 0.14588 0.029654 rpy=1.5708 0 -3.1416 -> xyz=0.078611 0.12644 0.029654 rpy=1.5708 0 -3.1416
- joint fr_wheel_joint: origin xyz=0.078747 -0.14712 0.029654 rpy=1.5708 0 0 -> xyz=0.078611 -0.12656 0.029654 rpy=1.5708 0 0
- joint joint_1: origin xyz=0.060647 -0.00061982 0.1296 rpy=0 0 0 -> xyz=0.060511 -5.5861E-05 0.0906 rpy=0 0 0
- joint joint_2: origin xyz=0.013741729606692 0.00180000000000001 0.0404532568712298 rpy=1.5707963267949 0 0 -> xyz=0.013742 0.0018 0.040453 rpy=1.5708 0 0
- joint joint_3: origin xyz=-0.0486912069159769 0.109677556359838 0 rpy=0 0 0 -> xyz=-0.048691 0.10968 0 rpy=0 0 0
- joint joint_4: origin xyz=0.0462467946124107 0.0790683813413976 -0.0104772836816603 rpy=-1.5707963267949 0 -0.530574095256852 -> xyz=0.046247 0.079068 -0.010477 rpy=-1.5708 0 -0.53057
- joint lidar_joint: origin xyz=0.045447 -0.074817 0.0658 rpy=0 0 0 -> xyz=-0.059689 -0.0002372 0.1148 rpy=0 0 0
- joint rgb_left_joint: axis 1 0 0 -> 0 0 0; origin xyz=0.0055995 0.0325 0.00355 rpy=0 0 0 -> xyz=0.005594 0.032538 0.00365 rpy=0 0 0
- joint rgb_left_optical_joint: axis 0 0 1 -> 0 0 0; origin xyz=0.0055995 0.0325 0.00355 rpy=-1.5708 0 -1.5708 -> xyz=0.005594 0.032538 0.00365 rpy=-1.5708 0 -1.5703

Commit message: Added basic arm manipulation feature

File: src/mobile_base_arm/urdf/mobile_base_arm.urdf (robot description, URDF)
Before this commit: robot mobile_base_arm, 21 links, 20 joints
Links:
- removed link bl_wheel_link
- removed link br_wheel_link
- removed link fl_wheel_link
- removed link fr_wheel_link
- removed link rgb_left_link
- removed link rgb_left_link_optical
- removed link rgb_right_link
- removed link rgb_right_link_optical
- added link bl_wheel, mass 0.041913; collision mesh filename=package://mobile_base_arm/meshes/bl_wheel.STL; visual mesh filename=package://mobile_base_arm/meshes/bl_wheel.STL
- added link br_wheel, mass 0.041913; collision mesh filename=package://mobile_base_arm/meshes/br_wheel.STL; visual mesh filename=package://mobile_base_arm/meshes/br_wheel.STL
- added link fl_wheel, mass 0.041913; collision mesh filename=package://mobile_base_arm/meshes/fl_wheel.STL; visual mesh filename=package://mobile_base_arm/meshes/fl_wheel.STL
- added link fr_wheel, mass 0.041913; collision mesh filename=package://mobile_base_arm/meshes/fr_wheel.STL; visual mesh filename=package://mobile_base_arm/meshes/fr_wheel.STL
- added link rpi_left, mass 0; collision mesh filename=package://mobile_base_arm/meshes/rpi_left.STL; visual mesh filename=package://mobile_base_arm/meshes/rpi_left.STL
- added link rpi_left_optical, mass 0; collision mesh filename=package://mobile_base_arm/meshes/rpi_left_optical.STL; visual mesh filename=package://mobile_base_arm/meshes/rpi_left_optical.STL
- added link rpi_right, mass 0; collision mesh filename=package://mobile_base_arm/meshes/rpi_right.STL; visual mesh filename=package://mobile_base_arm/meshes/rpi_right.STL
- added link rpi_right_optical, mass 0; collision mesh filename=package://mobile_base_arm/meshes/rpi_right_optical.STL; visual mesh filename=package://mobile_base_arm/meshes/rpi_right_optical.STL
- added link virtual_eef, mass 0.0071286; collision mesh filename=package://mobile_base_arm/meshes/virtual_eef.STL; visual mesh filename=package://mobile_base_arm/meshes/virtual_eef.STL
- link MPU9250_fl: mass 0.00062885 -> 0.00055422
- link camera_link: mass 0.0097885 -> 0
- link eef_link_1: mass 0.0096944 -> 0.0025659
Joints:
- removed joint MPU9250_fl_joint
- removed joint rgb_left_joint
- removed joint rgb_left_optical_joint
- removed joint rgb_right_joint
- removed joint rgb_right_optical_joint
- added joint MP9250_fl_joint: type fixed, parent base_link, child MPU9250_fl, origin xyz=0.082311 0.072761 0.05557 rpy=0 0 0, axis 0 0 0
- added joint rpi_left_joint: type fixed, parent camera_link, child rpi_left, origin xyz=0.005594 0.032538 0.00365 rpy=0 0 0, axis 0 0 0
- added joint rpi_left_optical_joint: type fixed, parent camera_link, child rpi_left_optical, origin xyz=0.005594 0.032538 0.00365 rpy=-1.5708 0 -1.5703, axis 0 0 0
- added joint rpi_right_joint: type fixed, parent camera_link, child rpi_right, origin xyz=0.0056 -0.0325 0.00355 rpy=0 0 0, axis 0 0 0
- added joint rpi_right_optical_joint: type fixed, parent camera_link, child rpi_right_optical, origin xyz=0.0056 -0.0325 0.00355 rpy=-1.5708 0 -1.5708, axis 0 0 0
- added joint virtual_eef_joint: type fixed, parent link_5, child virtual_eef, origin xyz=0.11861 0.0095012 -0.0036365 rpy=0 -1.5504 3.1099, axis 0 0 0
- joint bl_wheel_joint: child bl_wheel_link -> bl_wheel; origin xyz=-0.078589 0.12644 0.029654 rpy=1.5708 0 -3.1416 -> xyz=-0.078589 0.12644 0.011654 rpy=1.5708 0 -3.1416
- joint br_wheel_joint: child br_wheel_link -> br_wheel; origin xyz=-0.078589 -0.12656 0.029654 rpy=1.5708 0 0 -> xyz=-0.078589 -0.12656 0.011654 rpy=1.5708 0 0
- joint camera_joint: origin xyz=0.11151109677708 -5.58611123459007E-05 0.0299999999999999 rpy=0 0 0 -> xyz=0.11151 -5.5861E-05 0.012 rpy=0 0 0
- joint eef_finger_joint_2: mimic (none) -> joint=eef_finger_joint_1 multiplier=-1 offset=0
- joint eef_joint_1: origin xyz=0.038467 0.01414 -0.0179 rpy=-1.5708 0 3.1099 -> xyz=-0.012628 -0.0021 -0.080526 rpy=-1.5708 1.5504 0; parent link_5 -> virtual_eef
- joint eef_joint_2: mimic (none) -> joint=eef_joint_1 multiplier=-1 offset=0; origin xyz=0.038467 0.01414 0.009 rpy=-1.5708 0 3.1099 -> xyz=0.014267 -0.0021 -0.079979 rpy=-1.5708 1.5504 0; parent link_5 -> virtual_eef
- joint fl_wheel_joint: child fl_wheel_link -> fl_wheel; origin xyz=0.078611 0.12644 0.029654 rpy=1.5708 0 -3.1416 -> xyz=0.078611 0.12644 0.011654 rpy=1.5708 0 -3.1416
- joint fr_wheel_joint: child fr_wheel_link -> fr_wheel; origin xyz=0.078611 -0.12656 0.029654 rpy=1.5708 0 0 -> xyz=0.078611 -0.12656 0.011654 rpy=1.5708 0 0
- joint joint_1: limit lower=-3.1416 upper=3.1416 effort=0 velocity=0 -> lower=-2 upper=2 effort=0 velocity=0; origin xyz=0.060511 -5.5861E-05 0.0906 rpy=0 0 0 -> xyz=0.060511 -5.5861E-05 0.0726 rpy=0 0 0
- joint joint_4: origin xyz=0.046247 0.079068 -0.010477 rpy=-1.5708 0 -0.53057 -> xyz=0.050708 0.076451 -0.0107 rpy=-1.5708 0 -0.53057
- joint joint_5: origin xyz=0.00017223 -0.015127 0.028 rpy=1.5708 -1.5708 0 -> xyz=-0.005 -0.01535 0.028 rpy=1.5708 -1.5708 0
- joint lidar_joint: origin xyz=-0.059689 -0.0002372 0.1148 rpy=0 0 0 -> xyz=-0.059689 -0.0002372 0.0968 rpy=0 0 0

Commit message: Test D455

File: src/mobile_base_arm/urdf/mobile_base_arm.urdf (robot description, URDF)
Before this commit: robot mobile_base_arm, 22 links, 21 joints
Links:
- removed link MPU9250_fl
- removed link camera_link
- removed link rpi_left
- removed link rpi_left_optical
- removed link rpi_right
- removed link rpi_right_optical
- added link link_6, mass 0.015882; collision mesh filename=package://mobile_base_arm/meshes/link_6.STL; visual mesh filename=package://mobile_base_arm/meshes/link_6.STL
- link link_2: mass 0.098269 -> 0.064392
- link link_3: mass 0.084145 -> 0.050268
- link link_4: mass 0.023628 -> 0.016499
- link link_5: mass 0.02285 -> 0.021182
Joints:
- removed joint MP9250_fl_joint
- removed joint camera_joint
- removed joint rpi_left_joint
- removed joint rpi_left_optical_joint
- removed joint rpi_right_joint
- removed joint rpi_right_optical_joint
- added joint joint_6: type revolute, parent link_5, child link_6, origin xyz=0.0568500000006544 0.00510000000000022 0.0123999999969983 rpy=-1.57079632684769 0 -1.5707963267421, axis 0 0 -1, limit lower=-1.4 upper=1.4 effort=0 velocity=0
- joint eef_finger_joint_1: axis 0 0 0 -> 0 0 1; limit (none) -> lower=-1 upper=1 effort=0 velocity=0; mimic (none) -> joint=eef_joint_1 multiplier=-0.8 offset=0; origin xyz=-0.025075 0.017798 0.00135 rpy=0 0 0 -> xyz=0.025075 0.017798 0.00215 rpy=0 0 0; type fixed -> revolute
- joint eef_finger_joint_2: axis 0 0 0 -> 0 0 1; limit (none) -> lower=-1 upper=1 effort=0 velocity=0; mimic joint=eef_finger_joint_1 multiplier=-1 offset=0 -> joint=eef_joint_2 multiplier=-0.8 offset=0; origin xyz=-0.025013 -0.017886 0.00135 rpy=0 0 0 -> xyz=0.025013 -0.017886 0.00215 rpy=0 0 0; type fixed -> revolute
- joint eef_joint_1: axis 0 0 -1 -> 0 0 1; origin xyz=-0.012628 -0.0021 -0.080526 rpy=-1.5708 1.5504 0 -> xyz=-0.013659 -0.0021 -0.080358 rpy=-1.5708 -1.5633 -3.1416
- joint eef_joint_2: axis 0 0 -1 -> 0 0 1; origin xyz=0.014267 -0.0021 -0.079979 rpy=-1.5708 1.5504 0 -> xyz=0.01324 -0.0021 -0.080155 rpy=-1.5708 -1.5633 -3.1416
- joint joint_1: origin xyz=0.060511 -5.5861E-05 0.0726 rpy=0 0 0 -> xyz=0.059011 -5.5861E-05 0.0865 rpy=0 0 0
- joint joint_2: origin xyz=0.013742 0.0018 0.040453 rpy=1.5708 0 0 -> xyz=0.0137417296065389 0.0029000000007262 0.0415532568712299 rpy=1.5707963267949 0 0
- joint joint_3: axis 0 0 1 -> 0 0 -1; origin xyz=-0.048691 0.10968 0 rpy=0 0 0 -> xyz=-0.048691 0.10968 0 rpy=-3.1416 0 0
- joint joint_4: axis 0 0 1 -> 0 0 -1; origin xyz=0.050708 0.076451 -0.0107 rpy=-1.5708 0 -0.53057 -> xyz=0.0507079283195259 -0.0764510857051123 0.00960000000267675 rpy=1.57079632676818 0 0.530574095256852
- joint joint_5: axis 0 0 1 -> 0 0 -1; origin xyz=-0.005 -0.01535 0.028 rpy=1.5708 -1.5708 0 -> xyz=-0.00499999999999984 -0.01535 0.0294999999985077 rpy=1.57079632682587 -0.530574095256852 0
- joint lidar_joint: origin xyz=-0.059689 -0.0002372 0.0968 rpy=0 0 0 -> xyz=-0.059689 -0.0002372 0.1118 rpy=0 0 0
- joint virtual_eef_joint: origin xyz=0.11861 0.0095012 -0.0036365 rpy=0 -1.5504 3.1099 -> xyz=-0.00175 -0.00036346 0.13185 rpy=0 0.0075287 -1.5708; parent link_5 -> link_6
